Commit message: Add mobile base with LIDAR, shorten arm, and fix autonomous search-and-pick
Chassis + sensing:
- Enlarge base_link to a 0.38x0.26x0.08m box proportional to the wheelbase;
  keep base_link the kinematic root with base_footprint as a child.
- Add a front-mounted lidar_link + gpu_lidar sensor (270deg FOV, -135..135,
  publishing /scan), bridged in gazebo.launch.py.

Arm:
- Shorten all links 30% and taper radii; add sphere joint-caps for a cleaner
  look; introduce non-collinear shoulder/wrist offsets (like industrial arms)
  for better IK conditioning.

Autonomous search-and-pick (search_and_pick.py):
- Replace continuous spin with step-and-scan (rotate, stop, settle, capture)
  so detection is deterministic under sim load.
- Replace the two-pose search scheme, whose detection ranges no longer
  overlapped after the arm was shortened (leaving a ~[0.5,0.9]m dead zone the
  approach fell into), with a single wide search pose (pitch 25, detects
  [0.45,1.1]m) for spotting+approach, plus a steeper grasp-scan pose (pitch 38,
  [0.40,0.70]m) that run() uses to re-detect at the ~0.43m stop distance --
  which is within the shortened arm's ~0.45m grasp reach.
- Make the grasp-scan pose overridable via PickAndPlace.scan_position/pitch
  instead of module constants, so run() is reused unchanged.

Verified end-to-end: robot spins to find the box, tracks it smoothly from
1.14m to the stop distance, then grasps (box lifted to 0.14m), carries, and
places it -- PICK AND PLACE: DONE.

Co-Authored-By: Claude Opus 4.8 <noreply@anthropic.com>

File: src/pickplace_arm_description/urdf/pickplace_arm.gazebo.xacro (robot description, xacro)
@@ -136,3 +136,37 @@
     </sensor>
   </gazebo>
+  <!-- 2D LIDAR sensor (Gazebo Harmonic gpu_lidar) for SLAM + Nav2 -->
+  <gazebo reference="lidar_link">
+    <sensor name="lidar" type="gpu_lidar">
+      <topic>/scan</topic>
+      <update_rate>10</update_rate>
+      <always_on>1</always_on>
+      <visualize>true</visualize>
+      <lidar>
+        <scan>
+          <!-- 270 deg forward arc (-135..+135 deg); the excluded 90 deg
+               wedge points straight back at the arm, so the scan never hits
+               it. 270 samples keeps the same ~1 deg/sample resolution as a
+               360-sample full circle. -->
+          <horizontal>
+            <samples>270</samples>
+            <resolution>1</resolution>
+            <min_angle>-2.35619449</min_angle>
+            <max_angle>2.35619449</max_angle>
+          </horizontal>
+        </scan>
+        <range>
+          <min>0.12</min>
+          <max>8.0</max>
+          <resolution>0.01</resolution>
+        </range>
+        <noise>
+          <type>gaussian</type>
+          <mean>0.0</mean>
+          <stddev>0.01</stddev>
+        </noise>
+      </lidar>
+      <gz_frame_id>lidar_link</gz_frame_id>
+    </sensor>
+  </gazebo>
 </robot>

File: src/pickplace_arm_description/urdf/pickplace_arm.urdf.xacro (robot description, xacro)
@@ -9,6 +9,14 @@
   <!-- ============ Properties ============ -->
   <xacro:property name="PI" value="3.14159265359"/>
-  <xacro:property name="base_radius" value="0.08"/>
-  <xacro:property name="base_height" value="0.05"/>
+  <!-- Chassis is a box sized proportional to the wheelbase (wheels sit at
+       x=+/-0.12, y=+/-0.15). base_link origin is at wheel-axle height
+       (spawned at world z=0.05); box height 0.08 centered there spans world
+       z 0.01..0.09 so it clears the ground, and the arm still mounts on the
+       top face at z = base_height/2. base_radius is retained only as a
+       representative value for the inertia macro. -->
+  <xacro:property name="base_radius" value="0.13"/>
+  <xacro:property name="base_height" value="0.08"/>
+  <xacro:property name="base_length" value="0.38"/>
+  <xacro:property name="base_width" value="0.26"/>
   <!-- ============ Mobile base (4-wheel skid-steer) ============
        base_link is spawned at world z=0.05 (see gazebo.launch.py), which is
@@ -21,11 +29,43 @@
   <xacro:property name="wheel_x_offset" value="0.12"/>
   <xacro:property name="wheel_y_offset" value="0.15"/>
-  <xacro:property name="link1_len" value="0.15"/>
-  <xacro:property name="link2_len" value="0.30"/>
-  <xacro:property name="link3_len" value="0.25"/>
-  <xacro:property name="link4_len" value="0.10"/>
-  <xacro:property name="link5_len" value="0.08"/>
-  <xacro:property name="link6_len" value="0.06"/>
-  <xacro:property name="link_radius" value="0.035"/>
+  <!-- Arm link lengths trimmed 30% from the original (0.15/0.30/0.25/0.10/
+       0.08/0.06) for a more compact reach (~0.66m total vs ~0.94m before).
+       Radii are also tapered link-to-link (thicker at the shoulder, thinner
+       at the wrist) for a cleaner, more proportioned silhouette instead of
+       uniform-thickness segments; this and the joint-cap spheres below
+       are the "nicer looking" visual pass, built entirely from primitives
+       since no mesh-authoring tool (e.g. Blender) is available. -->
+  <xacro:property name="link1_len" value="0.105"/>
+  <xacro:property name="link2_len" value="0.21"/>
+  <xacro:property name="link3_len" value="0.175"/>
+  <xacro:property name="link4_len" value="0.07"/>
+  <xacro:property name="link5_len" value="0.056"/>
+  <xacro:property name="link6_len" value="0.042"/>
+  <!-- Lateral (forward, +x) offsets that break the arm out of a single
+       straight line, like real industrial arms (e.g. the UR series'
+       shoulder/wrist offsets). shoulder_offset kinks the upper arm forward
+       of the vertical base-yaw column; wrist_offset steps the wrist cluster
+       forward of the forearm. This avoids the fully-collinear home pose the
+       arm had before (which sat right on top of joint-axis alignments) and
+       gives cleaner IK conditioning near full extension. The J4-J5-J6 wrist
+       cluster itself is left un-offset so it stays a clean spherical wrist
+       for orientation control. Values re-verified reachable via compute_ik. -->
+  <xacro:property name="shoulder_offset" value="0.035"/>
+  <xacro:property name="wrist_offset" value="0.030"/>
+  <xacro:property name="link_radius" value="0.030"/>
+  <xacro:property name="link2_radius" value="0.032"/>
+  <xacro:property name="link3_radius" value="0.028"/>
+  <xacro:property name="link4_radius" value="0.026"/>
+  <xacro:property name="link5_radius" value="0.022"/>
+  <xacro:property name="link6_radius" value="0.022"/>
+  <!-- Joint-cap sphere radii (visual only, not collision; see each joint
+       below): slightly larger than the thicker of the two links they join,
+       so each pivot reads as a distinct actuator housing. -->
+  <xacro:property name="cap1_radius" value="0.045"/>
+  <xacro:property name="cap2_radius" value="0.040"/>
+  <xacro:property name="cap3_radius" value="0.035"/>
+  <xacro:property name="cap4_radius" value="0.032"/>
+  <xacro:property name="cap5_radius" value="0.028"/>
+  <xacro:property name="cap6_radius" value="0.026"/>
   <!-- Materials -->
   <material name="arm_orange"><color rgba="0.9 0.45 0.1 1.0"/></material>
@@ -42,15 +82,39 @@
     </inertial>
   </xacro:macro>
-  <!-- ============ Base Link ============ -->
+  <xacro:macro name="box_inertial" params="mass x y z">
+    <inertial>
+      <mass value="${mass}"/>
+      <inertia
+        ixx="${mass*(y*y+z*z)/12}" ixy="0.0" ixz="0.0"
+        iyy="${mass*(x*x+z*z)/12}" iyz="0.0"
+        izz="${mass*(x*x+y*y)/12}"/>
+    </inertial>
+  </xacro:macro>
+  <!-- ============ Base Link (box chassis, proportional to wheels) =======
+       base_link is the kinematic ROOT (as it was before the mobile base was
+       added), so MoveIt's world->base_link virtual joint and Cartesian path
+       planning work exactly as verified. base_footprint (Nav2's ground
+       projection frame) hangs off it as a CHILD below, rather than being the
+       root; making base_footprint the root broke MoveIt's planning tree
+       ("base_link and base_footprint not part of the same tree"). -->
   <link name="base_link">
     <visual>
-      <geometry><cylinder radius="${base_radius}" length="${base_height}"/></geometry>
-      <material name="arm_dark"/>
-    </visual>
-    <collision>
-      <geometry><cylinder radius="${base_radius}" length="${base_height}"/></geometry>
-    </collision>
-    <xacro:cylinder_inertial mass="2.0" radius="${base_radius}" length="${base_height}"/>
-  </link>
+      <geometry><box size="${base_length} ${base_width} ${base_height}"/></geometry>
+      <material name="arm_dark"/>
+    </visual>
+    <collision>
+      <geometry><box size="${base_length} ${base_width} ${base_height}"/></geometry>
+    </collision>
+    <xacro:box_inertial mass="2.0" x="${base_length}" y="${base_width}" z="${base_height}"/>
+  </link>
+  <!-- Nav2 ground-projection frame, as a child of base_link (base_link sits
+       one wheel-radius above the ground, so base_footprint is that far
+       below). -->
+  <link name="base_footprint"/>
+  <joint name="base_footprint_joint" type="fixed">
+    <parent link="base_link"/>
+    <child link="base_footprint"/>
+    <origin xyz="0 0 ${-wheel_radius}" rpy="0 0 0"/>
+  </joint>
   <!-- ============ Wheels (4-wheel skid-steer diff drive) ============
        Cylinder axis rotated onto Y so wheels roll about the Y axis (forward
@@ -81,6 +145,39 @@
   <xacro:wheel prefix="rear_left"   x_reflect="-1" y_reflect="1"/>
   <xacro:wheel prefix="rear_right"  x_reflect="-1" y_reflect="-1"/>
+  <!-- ============ 2D LIDAR (chassis-mounted, for SLAM/Nav2) ============
+       Mounted at the front edge of the chassis, ahead of both the
+       centrally-mounted arm (base at x=0) and the wrist RGB camera it
+       carries, so neither sits in the sensor's forward view. The scan
+       itself is restricted to a 270 deg forward arc in the Gazebo sensor
+       config (see pickplace_arm.gazebo.xacro) so the excluded 90 deg wedge
+       falls directly behind the sensor, exactly where the arm is,
+       instead of scanning through it. -->
+  <link name="lidar_link">
+    <visual>
+      <geometry><cylinder radius="0.03" length="0.04"/></geometry>
+      <material name="arm_grey"/>
+    </visual>
+    <collision>
+      <geometry><cylinder radius="0.03" length="0.04"/></geometry>
+    </collision>
+    <xacro:cylinder_inertial mass="0.1" radius="0.03" length="0.04"/>
+  </link>
+  <joint name="lidar_joint" type="fixed">
+    <parent link="base_link"/>
+    <child link="lidar_link"/>
+    <!-- inset from the front edge (chassis half-length 0.19, lidar radius
+         0.03 -> 0.02 m clearance) and mounted flush on the chassis top face
+         (top face at base_height/2=0.04, lidar half-length 0.02) so it sits
+         on the surface instead of floating above it. -->
+    <origin xyz="0.14 0 0.06" rpy="0 0 0"/>
+  </joint>
   <!-- ============ Link 1 (Shoulder Yaw) ============ -->
   <link name="link1">
+    <visual>
+      <!-- shoulder joint-cap: visual only, sits over joint1's pivot -->
+      <origin xyz="0 0 0" rpy="0 0 0"/>
+      <geometry><sphere radius="${cap1_radius}"/></geometry>
+      <material name="arm_dark"/>
+    </visual>
     <visual>
       <origin xyz="0 0 ${link1_len/2}" rpy="0 0 0"/>
@@ -104,18 +201,25 @@
   <link name="link2">
     <visual>
+      <!-- elbow-shoulder joint-cap: visual only, sits over joint2's pivot -->
+      <origin xyz="0 0 0" rpy="0 0 0"/>
+      <geometry><sphere radius="${cap2_radius}"/></geometry>
+      <material name="arm_dark"/>
+    </visual>
+    <visual>
       <origin xyz="0 0 ${link2_len/2}" rpy="0 0 0"/>
-      <geometry><box size="0.05 0.05 ${link2_len}"/></geometry>
+      <geometry><cylinder radius="${link2_radius}" length="${link2_len}"/></geometry>
       <material name="arm_grey"/>
     </visual>
     <collision>
       <origin xyz="0 0 ${link2_len/2}" rpy="0 0 0"/>
-      <geometry><box size="0.05 0.05 ${link2_len}"/></geometry>
-    </collision>
-    <xacro:cylinder_inertial mass="1.2" radius="0.04" length="${link2_len}"/>
+      <geometry><cylinder radius="${link2_radius}" length="${link2_len}"/></geometry>
+    </collision>
+    <xacro:cylinder_inertial mass="1.2" radius="${link2_radius}" length="${link2_len}"/>
   </link>
   <joint name="joint2" type="revolute">
     <parent link="link1"/>
     <child link="link2"/>
-    <origin xyz="0 0 ${link1_len}" rpy="0 0 0"/>
+    <!-- shoulder offset: upper arm steps forward of the base-yaw column -->
+    <origin xyz="${shoulder_offset} 0 ${link1_len}" rpy="0 0 0"/>
     <axis xyz="0 1 0"/>
     <limit lower="-${PI/2}" upper="${PI/2}" effort="50" velocity="1.5"/>
@@ -124,13 +228,19 @@
   <link name="link3">
     <visual>
+      <!-- elbow joint-cap: visual only, sits over joint3's pivot -->
+      <origin xyz="0 0 0" rpy="0 0 0"/>
+      <geometry><sphere radius="${cap3_radius}"/></geometry>
+      <material name="arm_dark"/>
+    </visual>
+    <visual>
       <origin xyz="0 0 ${link3_len/2}" rpy="0 0 0"/>
-      <geometry><box size="0.04 0.04 ${link3_len}"/></geometry>
+      <geometry><cylinder radius="${link3_radius}" length="${link3_len}"/></geometry>
       <material name="arm_orange"/>
     </visual>
     <collision>
       <origin xyz="0 0 ${link3_len/2}" rpy="0 0 0"/>
-      <geometry><box size="0.04 0.04 ${link3_len}"/></geometry>
-    </collision>
-    <xacro:cylinder_inertial mass="0.8" radius="0.03" length="${link3_len}"/>
+      <geometry><cylinder radius="${link3_radius}" length="${link3_len}"/></geometry>
+    </collision>
+    <xacro:cylinder_inertial mass="0.8" radius="${link3_radius}" length="${link3_len}"/>
   </link>
   <joint name="joint3" type="revolute">
@@ -144,18 +254,25 @@
   <link name="link4">
     <visual>
+      <!-- forearm-wrist joint-cap: visual only, sits over joint4's pivot -->
+      <origin xyz="0 0 0" rpy="0 0 0"/>
+      <geometry><sphere radius="${cap4_radius}"/></geometry>
+      <material name="arm_dark"/>
+    </visual>
+    <visual>
       <origin xyz="0 0 ${link4_len/2}" rpy="0 0 0"/>
-      <geometry><cylinder radius="0.03" length="${link4_len}"/></geometry>
+      <geometry><cylinder radius="${link4_radius}" length="${link4_len}"/></geometry>
       <material name="arm_grey"/>
     </visual>
     <collision>
       <origin xyz="0 0 ${link4_len/2}" rpy="0 0 0"/>
-      <geometry><cylinder radius="0.03" length="${link4_len}"/></geometry>
-    </collision>
-    <xacro:cylinder_inertial mass="0.4" radius="0.03" length="${link4_len}"/>
+      <geometry><cylinder radius="${link4_radius}" length="${link4_len}"/></geometry>
+    </collision>
+    <xacro:cylinder_inertial mass="0.4" radius="${link4_radius}" length="${link4_len}"/>
   </link>
   <joint name="joint4" type="revolute">
     <parent link="link3"/>
     <child link="link4"/>
-    <origin xyz="0 0 ${link3_len}" rpy="0 0 0"/>
+    <!-- wrist offset: wrist cluster steps forward of the forearm -->
+    <origin xyz="${wrist_offset} 0 ${link3_len}" rpy="0 0 0"/>
     <axis xyz="0 0 1"/>
     <limit lower="-${PI}" upper="${PI}" effort="20" velocity="2.0"/>
@@ -164,13 +281,19 @@
   <link name="link5">
     <visual>
+      <!-- wrist joint-cap: visual only, sits over joint5's pivot -->
+      <origin xyz="0 0 0" rpy="0 0 0"/>
+      <geometry><sphere radius="${cap5_radius}"/></geometry>
+      <material name="arm_dark"/>
+    </visual>
+    <visual>
       <origin xyz="0 0 ${link5_len/2}" rpy="0 0 0"/>
-      <geometry><cylinder radius="0.025" length="${link5_len}"/></geometry>
+      <geometry><cylinder radius="${link5_radius}" length="${link5_len}"/></geometry>
       <material name="arm_orange"/>
     </visual>
     <collision>
       <origin xyz="0 0 ${link5_len/2}" rpy="0 0 0"/>
-      <geometry><cylinder radius="0.025" length="${link5_len}"/></geometry>
-    </collision>
-    <xacro:cylinder_inertial mass="0.3" radius="0.025" length="${link5_len}"/>
+      <geometry><cylinder radius="${link5_radius}" length="${link5_len}"/></geometry>
+    </collision>
+    <xacro:cylinder_inertial mass="0.3" radius="${link5_radius}" length="${link5_len}"/>
   </link>
   <joint name="joint5" type="revolute">
@@ -184,13 +307,19 @@
   <link name="link6">
     <visual>
+      <!-- flange joint-cap: visual only, sits over joint6's pivot -->
+      <origin xyz="0 0 0" rpy="0 0 0"/>
+      <geometry><sphere radius="${cap6_radius}"/></geometry>
+      <material name="arm_grey"/>
+    </visual>
+    <visual>
       <origin xyz="0 0 ${link6_len/2}" rpy="0 0 0"/>
-      <geometry><cylinder radius="0.025" length="${link6_len}"/></geometry>
+      <geometry><cylinder radius="${link6_radius}" length="${link6_len}"/></geometry>
       <material name="arm_dark"/>
     </visual>
     <collision>
       <origin xyz="0 0 ${link6_len/2}" rpy="0 0 0"/>
-      <geometry><cylinder radius="0.025" length="${link6_len}"/></geometry>
-    </collision>
-    <xacro:cylinder_inertial mass="0.2" radius="0.025" length="${link6_len}"/>
+      <geometry><cylinder radius="${link6_radius}" length="${link6_len}"/></geometry>
+    </collision>
+    <xacro:cylinder_inertial mass="0.2" radius="${link6_radius}" length="${link6_len}"/>
   </link>
   <joint name="joint6" type="revolute">

Commit message: Fix skid-steer odometry with IMU/EKF fusion; complete SLAM+Nav2 verification
The 4-wheel skid-steer's wheel-only odometry drifted badly (heading error
from lateral scrub during turns), which distorted the SLAM map and made Nav2
goals miss. Fixed in layers, each verified against Gazebo ground truth:

- diff_drive_controller: open_loop -> false (integrate measured wheel
  velocities) and wheel_separation_multiplier 1.0 -> 1.46 (calibrated: odom
  rotation now matches physical within 1 deg; translation ratio 1.00).
- Added an IMU (imu_link + gz imu sensor + gz-sim-imu-system world plugin,
  bridged to /imu) and a robot_localization EKF (config/ekf.yaml) fusing wheel
  forward-velocity with IMU heading. diff_drive enable_odom_tf -> false so the
  EKF is the sole odom->base_link source. Result: odom error over a drive loop
  dropped from ~1.8 m / 90 deg to 0.08 m / 0 deg.

With good odometry, SLAM localization holds (0.66 m / 0 deg over a mapping
loop, vs 1.7-2.5 m before) and Nav2 navigates end-to-end: a NavigateToPose
goal plans a path, drives the base, steers around an obstacle (0.57 m
clearance) and arrives (status SUCCEEDED).

Nav2 config fixes for the installed (version-split) nav2 stack:
- bt_navigator: explicit plugin_lib_names excluding the route BT nodes, whose
  1.1.20 libs reference a ComputeAndTrackRoute action absent from the
  installed 1.1.18 nav2_msgs (undefined-symbol crash otherwise).
- Dropped twist_mux (its libdiagnostic_updater.so dependency is missing on
  this system); route controller_server cmd_vel straight to the diff drive
  controller since nav and visual-servo phases don't overlap.
- Tuned inflation_radius to 0.30 and slam_toolbox scan-matching for the
  small robot. Added wall/obstacle_box models for a test environment.

Co-Authored-By: Claude Opus 4.8 <noreply@anthropic.com>

File: src/pickplace_arm_description/urdf/pickplace_arm.gazebo.xacro (robot description, xacro)
@@ -170,3 +170,13 @@
     </sensor>
   </gazebo>
+  <!-- IMU sensor: publishes orientation + angular velocity, fused with wheel
+       odometry by the robot_localization EKF to keep heading accurate. -->
+  <gazebo reference="imu_link">
+    <sensor name="imu" type="imu">
+      <topic>/imu</topic>
+      <update_rate>50</update_rate>
+      <always_on>1</always_on>
+      <gz_frame_id>imu_link</gz_frame_id>
+    </sensor>
+  </gazebo>
 </robot>

File: src/pickplace_arm_description/urdf/pickplace_arm.urdf.xacro (robot description, xacro)
@@ -172,4 +172,19 @@
     <origin xyz="0.14 0 0.06" rpy="0 0 0"/>
   </joint>
+  <!-- IMU: its yaw is fused with the wheel odometry (robot_localization EKF)
+       to stabilize heading, which the 4-wheel skid-steer's wheel-only odom
+       estimates poorly (lateral scrub during turns causes heading drift that
+       corrupts SLAM). Mounted at the chassis center. -->
+  <link name="imu_link">
+    <inertial>
+      <mass value="0.02"/>
+      <inertia ixx="1e-6" ixy="0" ixz="0" iyy="1e-6" iyz="0" izz="1e-6"/>
+    </inertial>
+  </link>
+  <joint name="imu_joint" type="fixed">
+    <parent link="base_link"/>
+    <child link="imu_link"/>
+    <origin xyz="0 0 0.02" rpy="0 0 0"/>
+  </joint>
   <!-- ============ Link 1 (Shoulder Yaw) ============ -->
   <link name="link1">
