Commit message: Add warehouse world + front-facing RGB-D camera on the base
- worlds/warehouse.sdf: ~14x14 m world with outer walls, pillars, partial-wall
  corridors and crates (varied obstacles, navigable lanes). gazebo.launch.py
  now defaults to it (override via WORLD env var).
- Front RGB-D camera: front_camera_link on a short front mast pitched ~20 deg
  down; rgbd_camera sensor -> /front_camera; bridged /front_camera/{points,
  image,camera_info}. Detects the box ahead while the base drives (the wrist
  camera moves with the arm).

Verified: /scan sees the warehouse obstacles; /front_camera/points is organized
640x480 and a blue box 1.5 m ahead resolves to (1.48, 0.00, -0.02) in base_link.

Co-Authored-By: Claude Opus 4.8 <noreply@anthropic.com>

File: src/pickplace_arm_description/urdf/pickplace_arm.gazebo.xacro (robot description, xacro)
@@ -180,3 +180,30 @@
     </sensor>
   </gazebo>
+  <!-- Front RGB-D camera: detects the box ahead while the base drives. -->
+  <gazebo reference="front_camera_link">
+    <sensor name="front_rgbd_camera" type="rgbd_camera">
+      <topic>/front_camera</topic>
+      <update_rate>15</update_rate>
+      <always_on>1</always_on>
+      <visualize>true</visualize>
+      <camera>
+        <horizontal_fov>1.047</horizontal_fov>
+        <image>
+          <width>640</width>
+          <height>480</height>
+          <format>R8G8B8</format>
+        </image>
+        <clip>
+          <near>0.05</near>
+          <far>8.0</far>
+        </clip>
+        <noise>
+          <type>gaussian</type>
+          <mean>0.0</mean>
+          <stddev>0.007</stddev>
+        </noise>
+      </camera>
+      <gz_frame_id>front_camera_optical_link</gz_frame_id>
+    </sensor>
+  </gazebo>
 </robot>

File: src/pickplace_arm_description/urdf/pickplace_arm.urdf.xacro (robot description, xacro)
@@ -187,4 +187,31 @@
     <origin xyz="0 0 0.02" rpy="0 0 0"/>
   </joint>
+  <!-- Front-facing RGB-D camera on a short mast at the front of the chassis,
+       pitched ~20 deg down so its frustum sweeps the ground ~0.3-3 m ahead.
+       Used to detect the box while the base drives (the wrist camera moves
+       with the arm and can't watch ahead during navigation). -->
+  <link name="front_camera_link">
+    <visual>
+      <origin xyz="0 0 0" rpy="0 0 0"/>
+      <geometry><box size="0.03 0.06 0.03"/></geometry>
+      <material name="arm_dark"/>
+    </visual>
+    <collision>
+      <origin xyz="0 0 0" rpy="0 0 0"/>
+      <geometry><box size="0.03 0.06 0.03"/></geometry>
+    </collision>
+    <xacro:cylinder_inertial mass="0.05" radius="0.02" length="0.03"/>
+  </link>
+  <joint name="front_camera_joint" type="fixed">
+    <parent link="base_link"/>
+    <child link="front_camera_link"/>
+    <origin xyz="0.20 0 0.14" rpy="0 0.35 0"/>
+  </joint>
+  <link name="front_camera_optical_link"/>
+  <joint name="front_camera_optical_joint" type="fixed">
+    <parent link="front_camera_link"/>
+    <child link="front_camera_optical_link"/>
+    <origin xyz="0 0 0" rpy="-1.5708 0 -1.5708"/>
+  </joint>
   <!-- ============ Link 1 (Shoulder Yaw) ============ -->
   <link name="link1">
