Commit message: Fixed all the bugs for gazebo (migrated to harmonic)

File: src/pickplace_arm_description/urdf/pickplace_arm.gazebo.xacro (robot description, xacro)
@@ -49,5 +49,5 @@
   <!-- Gazebo Harmonic gz_ros2_control plugin -->
   <gazebo>
-    <plugin filename="gz_ros2_control-system" name="gz_ros2_control::GazeboSimROS2ControlPlugin">
+    <plugin filename="libgz_ros2_control-system.so" name="gz_ros2_control::GazeboSimROS2ControlPlugin">
       <parameters>$(find pickplace_arm_description)/config/arm_controllers.yaml</parameters>
       <ros>
@@ -56,3 +56,30 @@
     </plugin>
   </gazebo>
+  <!-- RGB-D Camera sensor (Gazebo Harmonic) -->
+  <gazebo reference="camera_link">
+    <sensor name="rgbd_camera" type="rgbd_camera">
+      <topic>/camera</topic>
+      <update_rate>30</update_rate>
+      <always_on>1</always_on>
+      <visualize>true</visualize>
+      <camera>
+        <horizontal_fov>1.047</horizontal_fov>
+        <image>
+          <width>640</width>
+          <height>480</height>
+          <format>R8G8B8</format>
+        </image>
+        <clip>
+          <near>0.05</near>
+          <far>5.0</far>
+        </clip>
+        <noise>
+          <type>gaussian</type>
+          <mean>0.0</mean>
+          <stddev>0.007</stddev>
+        </noise>
+      </camera>
+      <gz_frame_id>camera_optical_link</gz_frame_id>
+    </sensor>
+  </gazebo>
 </robot>

File: src/pickplace_arm_description/urdf/pickplace_arm.urdf.xacro (robot description, xacro)
@@ -1,4 +1,15 @@
 <?xml version="1.0"?>
 <robot name="pickplace_arm" xmlns:xacro="http://www.ros.org/wiki/xacro">
+  <!-- When true, pull in the Gazebo Harmonic ros2_control system + sensors.
+       Left false for the MoveIt/mock-hardware description so we don't end up
+       with two ros2_control systems. gazebo.launch.py sets this to true. -->
+  <xacro:arg name="use_gazebo" default="false"/>
+  <!-- Fix arm to world -->
+  <link name="world"/>
+  <joint name="world_joint" type="fixed">
+    <parent link="world"/>
+    <child link="base_link"/>
+    <origin xyz="0 0 0" rpy="0 0 0"/>
+  </joint>
   <!-- ============ Properties ============ -->
   <xacro:property name="PI" value="3.14159265359"/>
@@ -194,3 +205,31 @@
   <xacro:finger prefix="left" reflect="1"/>
   <xacro:finger prefix="right" reflect="-1"/>
+  <!-- ============ RGB-D Camera (mounted on gripper_base) ============ -->
+  <link name="camera_link">
+    <visual>
+      <origin xyz="0 0 0" rpy="0 0 0"/>
+      <geometry><box size="0.03 0.03 0.02"/></geometry>
+      <material name="arm_dark"/>
+    </visual>
+    <collision>
+      <origin xyz="0 0 0" rpy="0 0 0"/>
+      <geometry><box size="0.03 0.03 0.02"/></geometry>
+    </collision>
+    <xacro:cylinder_inertial mass="0.05" radius="0.015" length="0.02"/>
+  </link>
+  <joint name="camera_joint" type="fixed">
+    <parent link="gripper_base"/>
+    <child link="camera_link"/>
+    <origin xyz="0.04 0 0.02" rpy="0 0.5 0"/>
+  </joint>
+  <link name="camera_optical_link"/>
+  <joint name="camera_optical_joint" type="fixed">
+    <parent link="camera_link"/>
+    <child link="camera_optical_link"/>
+    <origin xyz="0 0 0" rpy="-1.5708 0 -1.5708"/>
+  </joint>
+  <!-- ============ Gazebo Harmonic integration (only when simulating) ============ -->
+  <xacro:if value="$(arg use_gazebo)">
+    <xacro:include filename="$(find pickplace_arm_description)/urdf/pickplace_arm.gazebo.xacro"/>
+  </xacro:if>
 </robot>

Commit message: Fixed the issue with picking the box

File: src/pickplace_arm_description/urdf/pickplace_arm.gazebo.xacro (robot description, xacro)
@@ -56,4 +56,22 @@
     </plugin>
   </gazebo>
+  <!-- High friction + soft contact on the finger pads so the gripper can
+       actually hold a box by friction in Gazebo Harmonic. -->
+  <gazebo reference="left_finger">
+    <mu1>2.0</mu1>
+    <mu2>2.0</mu2>
+    <kp>1e6</kp>
+    <kd>1.0</kd>
+    <minDepth>0.001</minDepth>
+    <maxVel>0.0</maxVel>
+  </gazebo>
+  <gazebo reference="right_finger">
+    <mu1>2.0</mu1>
+    <mu2>2.0</mu2>
+    <kp>1e6</kp>
+    <kd>1.0</kd>
+    <minDepth>0.001</minDepth>
+    <maxVel>0.0</maxVel>
+  </gazebo>
   <!-- RGB-D Camera sensor (Gazebo Harmonic) -->
   <gazebo reference="camera_link">

File: src/pickplace_arm_description/urdf/pickplace_arm.urdf.xacro (robot description, xacro)
@@ -199,5 +199,7 @@
       <child link="${prefix}_finger"/>
       <origin xyz="0 ${reflect*0.03} 0.045" rpy="0 0 0"/>
-      <axis xyz="0 1 0"/>
+      <!-- Mirror the axis per side so both fingers move outward together:
+           position 0 = closed (jaw gap 0.04 m), position 0.03 = open (gap 0.10 m) -->
+      <axis xyz="0 ${reflect} 0"/>
       <limit lower="0.0" upper="0.03" effort="20" velocity="0.1"/>
     </joint>

Commit message: 4 wheels

File: src/pickplace_arm_description/urdf/pickplace_arm.gazebo.xacro (robot description, xacro)
@@ -46,4 +46,24 @@
       <state_interface name="velocity"/>
     </joint>
+    <joint name="front_left_wheel_joint">
+      <command_interface name="velocity"/>
+      <state_interface name="position"/>
+      <state_interface name="velocity"/>
+    </joint>
+    <joint name="front_right_wheel_joint">
+      <command_interface name="velocity"/>
+      <state_interface name="position"/>
+      <state_interface name="velocity"/>
+    </joint>
+    <joint name="rear_left_wheel_joint">
+      <command_interface name="velocity"/>
+      <state_interface name="position"/>
+      <state_interface name="velocity"/>
+    </joint>
+    <joint name="rear_right_wheel_joint">
+      <command_interface name="velocity"/>
+      <state_interface name="position"/>
+      <state_interface name="velocity"/>
+    </joint>
   </ros2_control>
   <!-- Gazebo Harmonic gz_ros2_control plugin -->
@@ -74,4 +94,19 @@
     <maxVel>0.0</maxVel>
   </gazebo>
+  <!-- Wheel ground contact friction, enough traction to drive/skid-steer
+       without excessive slip. -->
+  <xacro:macro name="wheel_friction" params="link">
+    <gazebo reference="${link}">
+      <mu1>1.0</mu1>
+      <mu2>1.0</mu2>
+      <kp>1e6</kp>
+      <kd>1.0</kd>
+      <minDepth>0.001</minDepth>
+    </gazebo>
+  </xacro:macro>
+  <xacro:wheel_friction link="front_left_wheel"/>
+  <xacro:wheel_friction link="front_right_wheel"/>
+  <xacro:wheel_friction link="rear_left_wheel"/>
+  <xacro:wheel_friction link="rear_right_wheel"/>
   <!-- RGB-D Camera sensor (Gazebo Harmonic) -->
   <gazebo reference="camera_link">

File: src/pickplace_arm_description/urdf/pickplace_arm.urdf.xacro (robot description, xacro)
@@ -5,15 +5,20 @@
        with two ros2_control systems. gazebo.launch.py sets this to true. -->
   <xacro:arg name="use_gazebo" default="false"/>
-  <!-- Fix arm to world -->
-  <link name="world"/>
-  <joint name="world_joint" type="fixed">
-    <parent link="world"/>
-    <child link="base_link"/>
-    <origin xyz="0 0 0" rpy="0 0 0"/>
-  </joint>
+  <!-- base_link is the free-floating root: a mobile base (see wheels below)
+       carries it, rather than a fixed bolt to a "world" frame. -->
   <!-- ============ Properties ============ -->
   <xacro:property name="PI" value="3.14159265359"/>
   <xacro:property name="base_radius" value="0.08"/>
   <xacro:property name="base_height" value="0.05"/>
+  <!-- ============ Mobile base (4-wheel skid-steer) ============
+       base_link is spawned at world z=0.05 (see gazebo.launch.py), which is
+       unchanged by adding the base - wheel_radius is chosen to exactly
+       match that spawn height so the wheels touch the ground plane, and
+       every existing ground/grasp-height constant elsewhere in the repo
+       (pick_and_place.py, add_collision_box, etc.) stays valid untouched. -->
+  <xacro:property name="wheel_radius" value="0.05"/>
+  <xacro:property name="wheel_width" value="0.03"/>
+  <xacro:property name="wheel_x_offset" value="0.12"/>
+  <xacro:property name="wheel_y_offset" value="0.15"/>
   <xacro:property name="link1_len" value="0.15"/>
   <xacro:property name="link2_len" value="0.30"/>
@@ -48,4 +53,32 @@
     <xacro:cylinder_inertial mass="2.0" radius="${base_radius}" length="${base_height}"/>
   </link>
+  <!-- ============ Wheels (4-wheel skid-steer diff drive) ============
+       Cylinder axis rotated onto Y so wheels roll about the Y axis (forward
+       motion along X), matching the continuous joint axis "0 1 0" below. -->
+  <xacro:macro name="wheel" params="prefix x_reflect y_reflect">
+    <link name="${prefix}_wheel">
+      <visual>
+        <origin xyz="0 0 0" rpy="${PI/2} 0 0"/>
+        <geometry><cylinder radius="${wheel_radius}" length="${wheel_width}"/></geometry>
+        <material name="arm_dark"/>
+      </visual>
+      <collision>
+        <origin xyz="0 0 0" rpy="${PI/2} 0 0"/>
+        <geometry><cylinder radius="${wheel_radius}" length="${wheel_width}"/></geometry>
+      </collision>
+      <xacro:cylinder_inertial mass="0.3" radius="${wheel_radius}" length="${wheel_width}"/>
+    </link>
+    <joint name="${prefix}_wheel_joint" type="continuous">
+      <parent link="base_link"/>
+      <child link="${prefix}_wheel"/>
+      <origin xyz="${x_reflect*wheel_x_offset} ${y_reflect*wheel_y_offset} 0" rpy="0 0 0"/>
+      <axis xyz="0 1 0"/>
+      <dynamics damping="0.1" friction="0.05"/>
+    </joint>
+  </xacro:macro>
+  <xacro:wheel prefix="front_left"  x_reflect="1"  y_reflect="1"/>
+  <xacro:wheel prefix="front_right" x_reflect="1"  y_reflect="-1"/>
+  <xacro:wheel prefix="rear_left"   x_reflect="-1" y_reflect="1"/>
+  <xacro:wheel prefix="rear_right"  x_reflect="-1" y_reflect="-1"/>
   <!-- ============ Link 1 (Shoulder Yaw) ============ -->
   <link name="link1">

Commit message: Finalized corrections up to changing meshes

File: src/pickplace_arm_description/urdf/pickplace_arm.gazebo.xacro (robot description, xacro)
@@ -88,4 +88,48 @@
     </plugin>
   </gazebo>
+  <!-- Rigid grasp: weld the box to the gripper instead of relying on friction.
+       Friction alone was never reliable. The box slipped out mid-carry on
+       EVERY run of the Tugbot-warehouse mission (and intermittently before
+       that, which is what the raised mu values below were chasing). A
+       DetachableJoint per box gives a hard constraint that cannot slip
+       regardless of physics load, carry speed or how off-centre the grip is.
+       The gripper still physically closes on the box and the grasp is still
+       VERIFIED by the finger gap before anything attaches (see grab_below),
+       so this makes a confirmed grasp hold; it does not fake one.
+       parent_link is link6, NOT gripper_base, even though gripper_base is the
+       link every grasp pose is expressed in. Gazebo's URDF importer MERGES
+       links joined by fixed joints into their parent, so gripper_base does not
+       survive into the spawned SDF at all and naming it here fails the plugin
+       outright ("Link with name [gripper_base] not found in model
+       [pickplace_arm]. Failed to initialize."), silently leaving the box on
+       friction. link6 is what gripper_base was merged INTO, so it is the same
+       rigid body. Only links with a non-fixed joint (or a sensor) survive: to
+       check, run `gz model -m pickplace_arm` against a live sim and read the
+       link list. Verified empirically: attach/detach both work on link6.
+       Each box IS welded the moment it spawns, with no attach requested:
+       the plugin creates its joint as soon as the child model appears.
+       Verified by driving the base right after launch with nothing published,
+       and watching every box track the robot exactly (0.301 m for 0.301 m).
+       That makes the startup detach in PickAndPlace.__init__ load-bearing,
+       NOT a nicety: without it the robot tows all three boxes off the table
+       the moment it drives to the pick. Nothing moves between the box spawn
+       and the mission node starting, so issuing it there is soon enough. -->
+  <xacro:macro name="box_attach" params="color">
+    <gazebo>
+      <plugin filename="gz-sim-detachable-joint-system"
+              name="gz::sim::systems::DetachableJoint">
+        <parent_link>link6</parent_link>
+        <child_model>box_${color}</child_model>
+        <child_link>link</child_link>
+        <attach_topic>/box_${color}/attach</attach_topic>
+        <detach_topic>/box_${color}/detach</detach_topic>
+        <output_topic>/box_${color}/attach_state</output_topic>
+        <suppress_child_warning>true</suppress_child_warning>
+      </plugin>
+    </gazebo>
+  </xacro:macro>
+  <xacro:box_attach color="red"/>
+  <xacro:box_attach color="green"/>
+  <xacro:box_attach color="blue"/>
   <!-- High friction + soft contact on the finger pads so the gripper can
        actually hold a box by friction in Gazebo Harmonic. Raised 3.5 -> 5.0
