Commit message: Add MoveIt2 config, split Gazebo description, fix joint_limits types

File: src/pickplace_arm_description/urdf/pickplace_arm.urdf.xacro (robot description, xacro)
@@ -194,55 +194,3 @@
   <xacro:finger prefix="left" reflect="1"/>
   <xacro:finger prefix="right" reflect="-1"/>
-  <!-- ============ ros2_control ============ -->
-  <ros2_control name="pickplace_arm_system" type="system">
-    <hardware>
-      <plugin>gazebo_ros2_control/GazeboSystem</plugin>
-    </hardware>
-    <joint name="joint1">
-      <command_interface name="position"/>
-      <state_interface name="position"/>
-      <state_interface name="velocity"/>
-    </joint>
-    <joint name="joint2">
-      <command_interface name="position"/>
-      <state_interface name="position"/>
-      <state_interface name="velocity"/>
-    </joint>
-    <joint name="joint3">
-      <command_interface name="position"/>
-      <state_interface name="position"/>
-      <state_interface name="velocity"/>
-    </joint>
-    <joint name="joint4">
-      <command_interface name="position"/>
-      <state_interface name="position"/>
-      <state_interface name="velocity"/>
-    </joint>
-    <joint name="joint5">
-      <command_interface name="position"/>
-      <state_interface name="position"/>
-      <state_interface name="velocity"/>
-    </joint>
-    <joint name="joint6">
-      <command_interface name="position"/>
-      <state_interface name="position"/>
-      <state_interface name="velocity"/>
-    </joint>
-    <joint name="left_finger_joint">
-      <command_interface name="position"/>
-      <state_interface name="position"/>
-      <state_interface name="velocity"/>
-    </joint>
-    <joint name="right_finger_joint">
-      <command_interface name="position"/>
-      <state_interface name="position"/>
-      <state_interface name="velocity"/>
-    </joint>
-  </ros2_control>
-  <!-- ============ Gazebo ros2_control Plugin ============ -->
-  <gazebo>
-    <plugin name="gazebo_ros2_control" filename="libgazebo_ros2_control.so">
-      <parameters>$(find pickplace_arm_description)/config/arm_controllers.yaml</parameters>
-    </plugin>
-  </gazebo>
 </robot>

File: src/pickplace_arm_moveit_config/config/pickplace_arm.urdf.xacro (robot description, xacro)
@@ -2,4 +2,6 @@
 <robot xmlns:xacro="http://www.ros.org/wiki/xacro" name="pickplace_arm">
     <xacro:arg name="initial_positions_file" default="initial_positions.yaml" />
+    <!-- Use mock hardware, not Gazebo, when loaded by MoveIt -->
+    <xacro:arg name="use_gazebo" default="false" />
     <!-- Import pickplace_arm urdf file -->
     <xacro:include filename="$(find pickplace_arm_description)/urdf/pickplace_arm.urdf.xacro" />

Commit message: Front-face camera, cobra neutral pose, faster motion, robust final approach
- Front RGB-D camera moved onto the chassis front face (0.205,0,0.03, ~11 deg
  down) instead of floating on a mast; still detects the box accurately at
  1.0-2.5 m.
- Arm neutral/home pose is now a raised forward-curling "cobra" (HOME_CONFIG
  [0,0.30,0.40,0,0.45,0]) instead of straight up; used for the patrol tuck and
  the post-place home.
- Faster overall: Nav2 desired_linear_vel 0.35->0.55 + higher rotate/accel and
  velocity_smoother limits; diff_drive max lin 0.5->0.8, ang 1.5->2.2; arm
  max_velocity/accel 0.15->0.30.
- Final approach reworked (mission.servo_to_box): a two-phase visual servo --
  the FRONT camera (wide FOV, map-independent) drives the base straight in and
  centers the box, then the WRIST camera fine-servos to the grasp distance.
  Bounded left/right re-acquire sweep only (no full 360 spin, no blind forward
  drive that used to make the robot wander away), and a min forward-creep floor
  so it crosses the stop distance instead of stalling just outside it.

Verified end-to-end: patrol -> front-cam detect -> clean straight-in approach
-> pick -> deliver (-3.71,2.09) -> park (3.93,-3.93), MISSION DONE in ~113 s.

File: src/pickplace_arm_description/urdf/pickplace_arm.urdf.xacro (robot description, xacro)
@@ -187,8 +187,9 @@
     <origin xyz="0 0 0.02" rpy="0 0 0"/>
   </joint>
-  <!-- Front-facing RGB-D camera on a short mast at the front of the chassis,
-       pitched ~20 deg down so its frustum sweeps the ground ~0.3-3 m ahead.
-       Used to detect the box while the base drives (the wrist camera moves
-       with the arm and can't watch ahead during navigation). -->
+  <!-- Front-facing RGB-D camera mounted flush on the CHASSIS FRONT FACE
+       (the +x face is at base_length/2 = 0.19; the camera body is 0.03 deep so
+       its center sits at 0.19 + 0.015 = 0.205), near the top of the face and
+       centred in y. Pitched ~11 deg down so its frustum sweeps the ground
+       ahead for box detection while the base drives. -->
   <link name="front_camera_link">
     <visual>
@@ -206,5 +207,5 @@
     <parent link="base_link"/>
     <child link="front_camera_link"/>
-    <origin xyz="0.20 0 0.14" rpy="0 0.35 0"/>
+    <origin xyz="0.205 0 0.03" rpy="0 0.20 0"/>
   </joint>
   <link name="front_camera_optical_link"/>

Commit message: Optimal arm paths: stop the wrist unwinding ~2pi to the same orientation
Investigated the 'long useless arm paths'. It was NOT the optimizer or the DOF
count: measured wander ratio is ~1.0 (paths are already direct), and the arm is
a clean 6-DOF chain. The cause was the DOF RANGES -- the roll joints j1/j4/j6
were revolute with limits exactly [-pi, pi]. An angle near +pi and near -pi are
the SAME orientation, but a [-pi,pi] joint can't wrap, so reaching one from the
other unwinds the joint ~2pi the long way (measured: a move that should be 0.1
rad took 6.1 rad). The gripper-down grasp sits at j4 ~= +/-pi, so this bit hard.

Fix (keeps bounded revolute joints -- continuous joints break this MoveIt+KDL+
ros2_control stack with 2pi start-state aliasing and bad IK branches):
- Widen the roll joints j1/j4/j6 to [-2pi, 2pi] so the equivalent angle fits
  inside the limit (pickplace_arm.urdf.xacro).
- Normalize every commanded config's roll joints to the +/-2pi equivalent
  CLOSEST to the current angle (pick_and_place.py _normalize_roll_config,
  applied in move_config and the IK-seeded _move_pose_direct).

Verified: move_config to the opposite branch now travels 0.18 rad instead of
6.14; an arbitrary cross-pi reorientation dropped from 8.91 to 4.35 rad total;
all gripper-down mission poses move j4/j6 = 0.00 (no wrist spin); full mission
runs with 0 arm-move failures and a clean first-try claw grab.

File: src/pickplace_arm_description/urdf/pickplace_arm.urdf.xacro (robot description, xacro)
@@ -234,4 +234,8 @@
     <xacro:cylinder_inertial mass="1.0" radius="${link_radius}" length="${link1_len}"/>
   </link>
+  <!-- Roll joint with +/-2pi range (not +/-pi): a target near one pi limit can
+       then be reached from near the other via its +/-2pi equivalent (same
+       orientation) instead of unwinding ~2pi. Still bounded revolute, so no
+       continuous-joint state aliasing. -->
   <joint name="joint1" type="revolute">
     <parent link="base_link"/>
@@ -239,5 +243,5 @@
     <origin xyz="0 0 ${base_height/2}" rpy="0 0 0"/>
     <axis xyz="0 0 1"/>
-    <limit lower="-${PI}" upper="${PI}" effort="50" velocity="1.5"/>
+    <limit lower="-${2*PI}" upper="${2*PI}" effort="50" velocity="1.5"/>
   </joint>
   <!-- ============ Link 2 (Upper Arm Pitch) ============ -->
@@ -313,4 +317,6 @@
     <xacro:cylinder_inertial mass="0.4" radius="${link4_radius}" length="${link4_len}"/>
   </link>
+  <!-- Forearm roll with +/-2pi range so the gripper-down grasp (j4 ~= +/-pi) is
+       reachable from either side without a ~2pi unwind. -->
   <joint name="joint4" type="revolute">
     <parent link="link3"/>
@@ -319,5 +325,5 @@
     <origin xyz="${wrist_offset} 0 ${link3_len}" rpy="0 0 0"/>
     <axis xyz="0 0 1"/>
-    <limit lower="-${PI}" upper="${PI}" effort="20" velocity="2.0"/>
+    <limit lower="-${2*PI}" upper="${2*PI}" effort="20" velocity="2.0"/>
   </joint>
   <!-- ============ Link 5 (Wrist Pitch) ============ -->
@@ -366,4 +372,5 @@
     <xacro:cylinder_inertial mass="0.2" radius="${link6_radius}" length="${link6_len}"/>
   </link>
+  <!-- Wrist roll with +/-2pi range, same reason as j4. -->
   <joint name="joint6" type="revolute">
     <parent link="link5"/>
@@ -371,5 +378,5 @@
     <origin xyz="0 0 ${link5_len}" rpy="0 0 0"/>
     <axis xyz="0 0 1"/>
-    <limit lower="-${PI}" upper="${PI}" effort="10" velocity="2.0"/>
+    <limit lower="-${2*PI}" upper="${2*PI}" effort="10" velocity="2.0"/>
   </joint>
   <!-- ============ Gripper (simple 2-finger, mounted on link6) ============ -->

Commit message: Fixed the remaining issues (ready for v1)

File: src/pickplace_arm_description/urdf/pickplace_arm.urdf.xacro (robot description, xacro)
@@ -207,5 +207,11 @@
     <parent link="base_link"/>
     <child link="front_camera_link"/>
-    <origin xyz="0.205 0 0.03" rpy="0 0.20 0"/>
+    <!-- Zero rpy: the camera is rigidly aligned with base_link, so it always
+         points exactly along the chassis's own forward direction, with no
+         extra tilt to account for. Its wide 90deg horizontal FOV gives a
+         ~74deg vertical FOV; verify empirically (not just by this geometry
+         argument) that it still detects a table-height box from this mount
+         height at the distances the search/approach logic actually uses. -->
+    <origin xyz="0.205 0 0.01" rpy="0 0 0"/>
   </joint>
   <link name="front_camera_optical_link"/>
@@ -435,5 +441,15 @@
     <parent link="gripper_base"/>
     <child link="camera_link"/>
-    <origin xyz="0.04 0 0.02" rpy="0 0.5 0"/>
+    <!-- Zero rpy: the camera is rigidly aligned with gripper_base, so it
+         always looks exactly along the gripper's own local forward axis:
+         whatever the commanded arm orientation is, that is exactly what the
+         camera sees, with no extra per-camera tilt to compensate for.
+         Consequence: at zdown_quat (gripper pointing straight down, used for
+         grasp/carry/place) the camera looks purely horizontal, not downward,
+         so it cannot see anything below the gripper in that orientation.
+         Reading a tag or scanning for a box therefore needs the arm actually
+         pitched forward-down (scan_quat), not zdown; see SCAN_PITCH-style
+         constants in pick_and_place.py/search_and_pick.py/mission_2.py. -->
+    <origin xyz="0.04 0 0.01" rpy="0 0 0"/>
   </joint>
   <link name="camera_optical_link"/>

Commit message: Added mesh files for the lidar and cameras (RS-D435, RS-D405, SICK-TiM571) (placement needs more work)

File: src/pickplace_arm_description/urdf/pickplace_arm.urdf.xacro (robot description, xacro)
@@ -168,19 +168,43 @@
        so any ground-level box that SLAM/Nav2 used to see in the scan will no
        longer appear. -->
+  <!-- Modelled as a SICK TiM5xx (TiM571): a real 270 deg, single-plane scanner
+       whose datasheet geometry is what the sensor config above already
+       describes. Mesh referenced out of sick_scan_xd, not copied.
+       SICK's own URDF convention (sick_scan_xd/urdf/sick_scan.urdf.xacro):
+       the mesh is in METRES and its origin IS the laser centre, placed on the
+       link with no offset - so lidar_link sits exactly where the beams
+       originate, and the device body hangs around it. The body is 0.06 x 0.06
+       x 0.079 with the laser centre 0.05595 above its base plate, which is
+       what the mount joint below uses to stand it on the top plate. -->
   <link name="lidar_link">
     <visual>
-      <geometry><cylinder radius="0.03" length="0.04"/></geometry>
+      <geometry><mesh filename="package://sick_scan_xd/meshes/sick_tim_5xx.stl"/></geometry>
       <material name="arm_grey"/>
     </visual>
+    <!-- Collision is a PRIMITIVE, not the mesh, even though SICK's own URDF
+         reuses the mesh for both. A detailed triangle mesh is far more
+         expensive to collide than a box, and this housing never needs accurate
+         contact - it just has to exist. Using the mesh here measurably hurt:
+         the startup clock-jump count went from 0 to 1903 as the physics step
+         slowed. Box = the device envelope (0.06 x 0.06 x 0.079), centred
+         -0.01645 below the laser centre since the mesh origin IS that centre
+         and the body runs -0.05595..+0.02305 around it. -->
     <collision>
-      <geometry><cylinder radius="0.03" length="0.04"/></geometry>
+      <origin xyz="0 0 -0.01645" rpy="0 0 0"/>
+      <geometry><box size="0.06 0.06 0.079"/></geometry>
     </collision>
-    <xacro:cylinder_inertial mass="0.1" radius="0.03" length="0.04"/>
+    <xacro:cylinder_inertial mass="0.15" radius="0.03" length="0.079"/>
   </link>
   <joint name="lidar_joint" type="fixed">
     <parent link="top_plate_front_mount"/>
     <child link="lidar_link"/>
-    <!-- +z half the sensor body so it rests ON the plate, not half-sunk. -->
-    <origin xyz="0 0 0.02" rpy="0 0 0"/>
+    <!-- Stand the real device ON the plate: its base plate is 0.05595 below
+         the laser centre, and lidar_link IS the laser centre. This raises the
+         scan plane from 0.4037 to 0.4396 m above the floor (+0.036) versus the
+         placeholder cylinder - the price of modelling the actual sensor rather
+         than a puck. Nothing depends on the old value: warehouse walls span
+         the full height either way, and the carried box still rides 0.18 m
+         clear above the plane. -->
+    <origin xyz="0 0 0.05595" rpy="0 0 0"/>
   </joint>
   <!-- IMU: its yaw is fused with the wheel odometry (robot_localization EKF)
@@ -203,15 +227,28 @@
        face (at x=0.4937) and raised to look over the bumper line. Detects the
        box ahead while the base drives. -->
+  <!-- Modelled as an Intel RealSense D435 (87 deg HFOV, 0.05-10 m), the closest
+       real part to the 90 deg / 8 m sensor configured for it. Mesh referenced
+       out of realsense2_description, not copied.
+       Offsets copied from Intel's own _d435.urdf.xacro so the body sits
+       correctly around the frame: there, `<name>_link` is the DEPTH frame with
+       x forward - exactly the role front_camera_link plays here - and the mesh
+       is hung off it at (zero_depth_to_glass + glass_to_front, -cam_depth_py,
+       0) = (0.0043, -0.0175, 0) with rpy (pi/2, 0, pi/2). The -0.0175 y shift
+       is real: a D435's depth imager is not centred on its body, so the
+       housing renders offset from the optical axis. d435.dae is already in
+       metres (its COLLADA <unit> is 1.0), so no scale is applied.
+       front_camera_link itself has NOT moved - it stays at base_link
+       (0.5087, 0, 0.20), i.e. FRONT_CAM_Z = 0.332 m - because every detection
+       gate and the measured near-face bias are expressed against it. -->
   <link name="front_camera_link">
     <visual>
-      <origin xyz="0 0 0" rpy="0 0 0"/>
-      <geometry><box size="0.03 0.06 0.03"/></geometry>
-      <material name="arm_dark"/>
+      <origin xyz="0.0043 -0.0175 0" rpy="${PI/2} 0 ${PI/2}"/>
+      <geometry><mesh filename="package://realsense2_description/meshes/d435.dae"/></geometry>
     </visual>
     <collision>
-      <origin xyz="0 0 0" rpy="0 0 0"/>
-      <geometry><box size="0.03 0.06 0.03"/></geometry>
+      <origin xyz="0 -0.0175 0" rpy="0 0 0"/>
+      <geometry><box size="0.02505 0.090 0.025"/></geometry>
     </collision>
-    <xacro:cylinder_inertial mass="0.05" radius="0.02" length="0.03"/>
+    <xacro:cylinder_inertial mass="0.072" radius="0.02" length="0.025"/>
   </link>
   <joint name="front_camera_joint" type="fixed">
@@ -243,20 +280,38 @@
        straight down the camera looks straight down too, so scanning for a box
        or reading a tag needs the arm actually pitched to a scan pose. -->
+  <!-- Modelled as an Intel RealSense D405: the short-range part of the family,
+       built for exactly this eye-in-hand job (60 deg HFOV, useful from a few
+       mm out), which matches the 60 deg / 0.05-5 m sensor configured for it.
+       Mesh referenced out of realsense2_description, not copied.
+       Offsets copied from Intel's _d405.urdf.xacro, same convention as the
+       D435 above: mesh at (zero_depth_to_glass + glass_to_front, -cam_depth_py,
+       0) = (0.0038, -0.009, 0), rpy (pi/2, 0, pi/2). Unlike d435.dae, d405.stl
+       is authored in MILLIMETRES, so it needs the 0.001 scale Intel applies. -->
   <link name="camera_link">
     <visual>
-      <origin xyz="0 0 0" rpy="0 0 0"/>
-      <geometry><box size="0.03 0.03 0.02"/></geometry>
+      <origin xyz="0.0038 -0.009 0" rpy="${PI/2} 0 ${PI/2}"/>
+      <geometry>
+        <mesh filename="package://realsense2_description/meshes/d405.stl"
+              scale="0.001 0.001 0.001"/>
+      </geometry>
       <material name="arm_dark"/>
     </visual>
     <collision>
-      <origin xyz="0 0 0" rpy="0 0 0"/>
-      <geometry><box size="0.03 0.03 0.02"/></geometry>
+      <origin xyz="-0.0078 -0.009 0" rpy="0 0 0"/>
+      <geometry><box size="0.023 0.042 0.042"/></geometry>
     </collision>
-    <xacro:cylinder_inertial mass="0.05" radius="0.015" length="0.02"/>
+    <xacro:cylinder_inertial mass="0.045" radius="0.021" length="0.023"/>
   </link>
   <joint name="camera_joint" type="fixed">
     <parent link="fr3_hand"/>
     <child link="camera_link"/>
-    <origin xyz="0.055 0 0.04" rpy="0 -1.5708 0"/>
+    <!-- Moved out 0.055 -> 0.068 along the hand's x. The real D405 is 42 mm
+         square where the placeholder box was 30x20, and fr3_hand's collision
+         capsule has a 0.04 m radius about the hand axis - at 0.055 the real
+         body would visibly clip into the hand. 0.068 puts its nearest face
+         0.047 m off the axis, clear of the capsule, without touching the
+         approach-axis alignment (this offset is perpendicular to the view
+         direction, and detection transforms through TF regardless). -->
+    <origin xyz="0.068 0 0.04" rpy="0 -1.5708 0"/>
   </joint>
   <link name="camera_optical_link"/>
