Commit message: Fixed the remaining issues with the placement of the sensors

File: src/pickplace_arm_description/urdf/pickplace_arm.urdf.xacro (robot description, xacro)
@@ -78,4 +78,55 @@
   <xacro:include filename="$(find clearpath_platform_description)/urdf/a200/a200.urdf.xacro"/>
   <xacro:include filename="$(find clearpath_platform_description)/urdf/a200/attachments/top_plate.urdf.xacro"/>
+  <!-- ============ Wheel visual override ============
+       WHY THIS EXISTS: Clearpath's wheel.dae is a 7 inch-radius (0.1778 m)
+       tyre, but every other number in the A200 says the wheel is 6.5 inch
+       (0.1651 m) - the collision cylinder (`wheel_radius`), the controller's
+       `wheel_diameter` 0.3302, and `wheel_vertical_offset` 0.03282, which is
+       what puts base_footprint exactly 0.1651 under the axle. Physics rests the
+       COLLISION cylinder on the floor, so the 12.7 mm-larger visual mesh sank
+       that far into the ground on all four wheels.
+       Scaling the mesh by 0.1651/0.1778 = 0.9285714 in its two RADIAL axes
+       (x and z; the mesh's y is the axle, and already spans exactly the 0.1143
+       `wheel_length`) makes the rendered tyre agree with the cylinder it
+       actually rolls on. Nothing kinematic changes - the collision, the joint
+       origins and base_footprint are untouched, so GROUND_Z (-0.13228) and the
+       odometry stay exactly as they were.
+       WHY IT IS HERE AND NOT IN wheel.urdf.xacro: clearpath_common is a nested
+       git checkout, not part of this repo's history, so an edit there would be
+       invisible to review and lost on any re-clone. Redefining the macro after
+       the include but BEFORE the <xacro:a200> call means xacro resolves
+       a200_wheel to THIS definition when it expands the a200 body - the fix
+       lives in our own tracked package and upstream stays pristine.
+       The body below mirrors Clearpath's macro exactly apart from the mesh
+       scale. The two dimensions are inlined as literals rather than read from
+       ${wheel_radius}/${wheel_length}, because those properties are declared
+       inside the `a200` macro and are not in scope for a macro defined out
+       here. -->
+  <xacro:macro name="a200_wheel" params="wheel_prefix *joint_pose">
+    <link name="${wheel_prefix}_wheel">
+      <inertial>
+        <mass value="2.637"/>
+        <origin xyz="0 0 0"/>
+        <inertia ixx="0.02467" ixy="0" ixz="0" iyy="0.04411" iyz="0" izz="0.02467"/>
+      </inertial>
+      <visual>
+        <origin xyz="0 0 0" rpy="0 0 0"/>
+        <geometry>
+          <mesh filename="package://clearpath_platform_description/meshes/a200/wheel.dae"
+                scale="0.9285714 1.0 0.9285714"/>
+        </geometry>
+      </visual>
+      <collision>
+        <origin xyz="0 0 0" rpy="${PI/2} 0 0"/>
+        <geometry><cylinder length="0.1143" radius="0.1651"/></geometry>
+      </collision>
+    </link>
+    <joint name="${wheel_prefix}_wheel_joint" type="continuous">
+      <parent link="base_link"/>
+      <child link="${wheel_prefix}_wheel"/>
+      <xacro:insert_block name="joint_pose"/>
+      <axis xyz="0 1 0" rpy="0 0 0"/>
+    </joint>
+  </xacro:macro>
   <xacro:a200 wheel="default"/>
   <!-- Standard user-rail top plate on the A200's default_mount. This is what
@@ -250,43 +301,56 @@
        curves away). front_bumper_mount is 1.6 mm proud of it at z=0.091, i.e.
        squarely in the middle of the flat region - so mounting with no z offset
-       puts the camera body at z 0.0785..0.1035, entirely on the panel. -->
-  <!-- Modelled as an Intel RealSense D435 (87 deg HFOV, 0.05-10 m), the closest
-       real part to the 90 deg / 8 m sensor configured for it. Mesh referenced
-       out of realsense2_description, not copied.
-       Offsets copied from Intel's own _d435.urdf.xacro so the body sits
-       correctly around the frame: there, `<name>_link` is the DEPTH frame with
-       x forward - exactly the role front_camera_link plays here - and the mesh
-       is hung off it at (zero_depth_to_glass + glass_to_front, -cam_depth_py,
-       0) = (0.0043, -0.0175, 0) with rpy (pi/2, 0, pi/2). The -0.0175 y shift
-       is real: a D435's depth imager is not centred on its body, so the
-       housing renders offset from the optical axis. d435.dae is already in
-       metres (its COLLADA <unit> is 1.0), so no scale is applied.
-       That mesh + origin + rpy resolve to a body occupying, in this link's
-       frame, x -0.02075..+0.0043, y -0.06241..+0.0275, z -0.0125..+0.0125:
-       the back face is 20.75 mm BEHIND the link and the front glass 4.3 mm
-       ahead of it. Those two numbers are what the mount joint's x is set from.
-       THE MATERIAL IS NOT COSMETIC. d435.dae carries exactly one material - a
-       lambert with diffuse 0.749 grey and no ambient/specular - and with no
-       <material> here that is what Gazebo renders, which under the sim's
-       lighting reads as a plain WHITE block. An explicit URDF material is
-       converted into an SDF <material> that overrides the mesh's own, so this
-       is what makes the housing look like the dark camera it is, matching the
-       wrist D405 below. -->
+       puts the camera body at z 0.0765..0.1055, entirely on the panel. -->
+  <!-- Modelled as an Intel RealSense D455 (87 x 58 deg FOV), which matches the
+       90 deg / 8 m sensor configured for it and is the D400-series part
+       normally fitted to a mobile base. Mesh referenced out of
+       realsense2_description, not copied.
+       IT IS A D455 AND NOT A D435 FOR A RENDERING REASON, measured not assumed.
+       Gazebo (gz-sim 8.14, ogre2) IGNORES an SDF <material> on a mesh that
+       carries its own embedded materials, and d435.dae carries exactly one - a
+       lambert with diffuse 0.749 and no ambient/specular, which saturates to
+       plain WHITE under the sim's lighting. That is not a theory: rendering
+       d435.dae twice side by side, once bare and once with an SDF material
+       forced to pure RED, produced two identical white bars, while d405.stl
+       with a forced BLUE came out blue. An STL carries no material, so the
+       <material> below is the only thing describing it and Gazebo honours it.
+       d455.stl is the closest STL in the family - and at 2.5 MB against
+       d435.dae's 15 MB it is markedly cheaper to load and draw as well.
+       Offsets follow Intel's own _d455.urdf.xacro: the mesh is authored in
+       MILLIMETRES (hence scale 0.001) with its origin at the front plate, hung
+       off the link with rpy (pi/2, 0, pi/2) and x = zero_depth_to_glass +
+       glass_to_front = 0.00455 + 0.0001.
+       ONE DELIBERATE DEVIATION: Intel also shifts the mesh by -cam_depth_py
+       (-0.0475), because d455.stl's origin is the housing's lateral CENTRE and
+       that shift is what lands the real depth module on the link. Applying it
+       would hang a 124 mm bar almost entirely off one side of the robot's
+       centreline (y -0.1095..+0.0145). Since front_camera_link is a frame we
+       define, and the sim renders from wherever front_camera_optical_link is
+       put, nothing functional depends on reproducing the D455's internal
+       optical offset - so the shift is dropped and the housing is centred on
+       the chassis, the way one would actually bolt it on.
+       Mesh + origin + rpy therefore resolve to a body occupying, in this
+       link's frame, x -0.02135..+0.00465, y -0.062..+0.062, z -0.0145..+0.0145:
+       the back face is 21.35 mm BEHIND the link and the front glass 4.65 mm
+       ahead of it. Those are what the mount joint's x is set from. -->
   <link name="front_camera_link">
     <visual>
-      <origin xyz="0.0043 -0.0175 0" rpy="${PI/2} 0 ${PI/2}"/>
-      <geometry><mesh filename="package://realsense2_description/meshes/d435.dae"/></geometry>
-      <material name="arm_dark"/>
+      <origin xyz="0.00465 0 0" rpy="${PI/2} 0 ${PI/2}"/>
+      <geometry>
+        <mesh filename="package://realsense2_description/meshes/d455.stl"
+              scale="0.001 0.001 0.001"/>
+      </geometry>
+      <material name="arm_grey"/>
     </visual>
-    <!-- Box = the mesh envelope above. Its x origin was 0, which centred the
-         box on the link and so pushed its back face 12.5 mm behind the real
-         housing - harmless while the camera floated in mid-air, but now that
-         the housing is flush against the panel that phantom 8 mm would sit
-         inside the chassis. -0.00823 is the true envelope centre. -->
+    <!-- Box = the mesh envelope above (0.026 x 0.124 x 0.029), centred on that
+         envelope rather than on the link. Centring it on the link instead
+         would push its back face 8 mm behind the real housing, which now that
+         the camera is bedded against the panel would put phantom collision
+         geometry inside the chassis. -->
     <collision>
-      <origin xyz="-0.00823 -0.0175 0" rpy="0 0 0"/>
-      <geometry><box size="0.02505 0.090 0.025"/></geometry>
+      <origin xyz="-0.00835 0 0" rpy="0 0 0"/>
+      <geometry><box size="0.026 0.124 0.029"/></geometry>
     </collision>
-    <xacro:cylinder_inertial mass="0.072" radius="0.02" length="0.025"/>
+    <xacro:cylinder_inertial mass="0.072" radius="0.02" length="0.026"/>
   </link>
   <joint name="front_camera_joint" type="fixed">
@@ -300,5 +364,5 @@
          while the camera frame's z is world-up. Do not add a tilt here.
          x = +0.019 seats the housing ON the panel: the back face lands at
-         base_link 0.40425 against the panel's 0.4044, so it beds in by 0.15 mm
+         base_link 0.40365 against the panel's 0.4044, so it beds in by 0.75 mm
          with no gap to show. It was +0.1027, which left the back face at
          0.48795 - 83 mm of clear air in front of the chassis - and z was
@@ -347,5 +411,5 @@
               scale="0.001 0.001 0.001"/>
       </geometry>
-      <material name="arm_dark"/>
+      <material name="arm_grey"/>
     </visual>
     <collision>
@@ -358,24 +422,29 @@
     <parent link="fr3_hand"/>
     <child link="camera_link"/>
-    <!-- x = 0.048 seats the D405 against the hand. It was 0.068, chosen to
-         clear a 0.04 m collision CAPSULE about the hand axis - but that capsule
-         only exists when with_sc=true, and franka_robot is called above with
-         with_sc="false", so nothing was ever there to clear. The hand's real
-         surface is much closer in: hand.stl's side face is a TAPER, measured by
-         cross-sectioning the mesh at the camera's own y band -
+    <!-- x = 0.043 seats the D405 against the hand with NO GAP ANYWHERE. It was
+         0.068, chosen to clear a 0.04 m collision CAPSULE about the hand axis -
+         but that capsule only exists when with_sc=true, and franka_robot is
+         called above with with_sc="false", so nothing was ever there to clear.
+         The hand's side is not a flat face, it is a TAPER, measured by
+         cross-sectioning hand.stl at the camera's own y band:
              hand z 0.021 -> x 0.0280      hand z 0.044 -> x 0.0223
-         (widest at 0.0315 down near z=0.005, narrowing all the way up).
-         With the mesh reaching 0.021 back from camera_link, x=0.068 put the
-         camera's back face at hand x=0.047, leaving 19 mm of visible air
-         between it and the hand.
-         0.048 puts that back face at 0.027, which beds 1 mm into the hand at
-         the camera's lower edge and leaves ~4 mm at its upper edge where the
-         taper has fallen away - flush to the eye, and the small bite guarantees
-         no daylight shows through. This offset is perpendicular to the view
-         direction and does not touch the approach-axis alignment; detections
-         transform through TF regardless. camera_link vs fr3_hand is already
+         (widest at 0.0315 near z=0.005, narrowing all the way up). The camera
+         body spans hand z 0.0208..0.0438, so the surface it has to meet slides
+         inward by 5.7 mm from its bottom edge to its top.
+         With the mesh reaching 0.021 back from camera_link, x=0.068 left the
+         back face at hand x=0.047 - 19 mm of open air. An intermediate 0.048
+         put it at 0.027, which touched at the BOTTOM edge but still left ~4 mm
+         showing at the top, where the taper had fallen away: the gap that was
+         still visible. Seating it against the NARROWEST point of the contact
+         band instead (0.0223 at the top edge) is what closes it: 0.043 puts the
+         back face at 0.022, so the housing meets or bites into the hand over
+         the whole band - 0.3 mm proud at the top, 6 mm buried at the bottom.
+         The buried part is inside a solid link and never shows.
+         This offset is perpendicular to the view direction and does not touch
+         the approach-axis alignment; detections transform through TF
+         regardless. camera_link vs fr3_hand is already
          disable_collisions="Adjacent" in the SRDF, so the contact costs
          nothing in planning. -->
-    <origin xyz="0.048 0 0.04" rpy="0 -1.5708 0"/>
+    <origin xyz="0.043 0 0.04" rpy="0 -1.5708 0"/>
   </joint>
   <link name="camera_optical_link"/>

Commit message: Cleaned up the workspace

File: src/pickplace_arm_description/urdf/pickplace_arm.urdf.xacro (robot description, xacro)
@@ -5,8 +5,12 @@
   <!-- Franka Hand gripper.                                                  -->
   <!--                                                                       -->
-  <!-- Base and arm are REFERENCED out of the upstream description packages  -->
-  <!-- via $(find ...), never copied, so their meshes stay in one place:      -->
+  <!-- Base and arm geometry is VENDORED into this package, under            -->
+  <!-- urdf/vendor/ and meshes/. It used to be referenced via $(find ...) out -->
+  <!-- of the upstream packages, but those were nested git checkouts that     -->
+  <!-- could not be pushed with this project, so the subset this robot        -->
+  <!-- actually uses was copied in and the URIs repointed. Provenance:        -->
   <!--   * clearpath_platform_description (humble)  -> Husky A200            -->
   <!--   * franka_description 1.6.1                 -> FR3 arm + Franka Hand -->
+  <!-- Upstream licences are kept beside the meshes as LICENSE.<package>.     -->
   <!--                                                                       -->
   <!-- NOTE on the Husky variant: the A300 does NOT exist on clearpath_common -->
@@ -76,6 +80,6 @@
          wheels       x +/-0.256, y +/-0.2775, radius 0.1651, track 0.555
          default_mount   z = 0.224 -->
-  <xacro:include filename="$(find clearpath_platform_description)/urdf/a200/a200.urdf.xacro"/>
-  <xacro:include filename="$(find clearpath_platform_description)/urdf/a200/attachments/top_plate.urdf.xacro"/>
+  <xacro:include filename="$(find pickplace_arm_description)/urdf/vendor/a200/a200.urdf.xacro"/>
+  <xacro:include filename="$(find pickplace_arm_description)/urdf/vendor/a200/attachments/top_plate.urdf.xacro"/>
   <!-- ============ Wheel visual override ============
        WHY THIS EXISTS: Clearpath's wheel.dae is a 7 inch-radius (0.1778 m)
@@ -92,10 +96,13 @@
        origins and base_footprint are untouched, so GROUND_Z (-0.13228) and the
        odometry stay exactly as they were.
-       WHY IT IS HERE AND NOT IN wheel.urdf.xacro: clearpath_common is a nested
-       git checkout, not part of this repo's history, so an edit there would be
-       invisible to review and lost on any re-clone. Redefining the macro after
-       the include but BEFORE the <xacro:a200> call means xacro resolves
-       a200_wheel to THIS definition when it expands the a200 body - the fix
-       lives in our own tracked package and upstream stays pristine.
+       WHY IT IS HERE AND NOT IN wheel.urdf.xacro: originally because
+       clearpath_common was a nested git checkout whose edits would have been
+       lost on any re-clone. That package is gone now and wheel.urdf.xacro is
+       vendored under urdf/vendor/, so the fix COULD be applied there - it is
+       deliberately not, so the vendored files stay a faithful copy of upstream
+       apart from mechanical path rewrites. Anything this project changes about
+       the A200 lives here, where it is visible next to the reasoning.
+       Redefining the macro after the include but BEFORE the <xacro:a200> call
+       is what makes xacro resolve a200_wheel to THIS definition.
        The body below mirrors Clearpath's macro exactly apart from the mesh
        scale. The two dimensions are inlined as literals rather than read from
@@ -113,5 +120,5 @@
         <origin xyz="0 0 0" rpy="0 0 0"/>
         <geometry>
-          <mesh filename="package://clearpath_platform_description/meshes/a200/wheel.dae"
+          <mesh filename="package://pickplace_arm_description/meshes/a200/wheel.dae"
                 scale="0.9285714 1.0 0.9285714"/>
         </geometry>
@@ -167,13 +174,13 @@
                                   MoveIt uses the real collision meshes.
          ros2_control="false"  -> ditto, our own block owns the interfaces. -->
-  <xacro:include filename="$(find franka_description)/robots/common/franka_robot.xacro"/>
+  <xacro:include filename="$(find pickplace_arm_description)/urdf/vendor/franka/robots/common/franka_robot.xacro"/>
   <xacro:franka_robot
     robot_type="fr3"
     arm_prefix=""
     no_prefix="false"
-    joint_limits="${xacro.load_yaml('$(find franka_description)/robots/fr3/joint_limits.yaml')}"
-    inertials="${xacro.load_yaml('$(find franka_description)/robots/fr3/inertials.yaml')}"
-    kinematics="${xacro.load_yaml('$(find franka_description)/robots/fr3/kinematics.yaml')}"
-    dynamics="${xacro.load_yaml('$(find franka_description)/robots/fr3/dynamics.yaml')}"
+    joint_limits="${xacro.load_yaml('$(find pickplace_arm_description)/config/franka/fr3/joint_limits.yaml')}"
+    inertials="${xacro.load_yaml('$(find pickplace_arm_description)/config/franka/fr3/inertials.yaml')}"
+    kinematics="${xacro.load_yaml('$(find pickplace_arm_description)/config/franka/fr3/kinematics.yaml')}"
+    dynamics="${xacro.load_yaml('$(find pickplace_arm_description)/config/franka/fr3/dynamics.yaml')}"
     accelerometer_config="none"
     hand="true"
@@ -221,5 +228,5 @@
   <!-- Modelled as a SICK TiM5xx (TiM571): a real 270 deg, single-plane scanner
        whose datasheet geometry is what the sensor config above already
-       describes. Mesh referenced out of sick_scan_xd, not copied.
+       describes. Mesh vendored from sick_scan_xd into meshes/sensors/.
        SICK's own URDF convention (sick_scan_xd/urdf/sick_scan.urdf.xacro):
        the mesh is in METRES and its origin IS the laser centre, placed on the
@@ -238,5 +245,5 @@
   <link name="lidar_link">
     <visual>
-      <geometry><mesh filename="package://sick_scan_xd/meshes/sick_tim_5xx.stl"/></geometry>
+      <geometry><mesh filename="package://pickplace_arm_description/meshes/sensors/sick_tim_5xx.stl"/></geometry>
       <material name="arm_grey"/>
     </visual>
@@ -304,6 +311,6 @@
   <!-- Modelled as an Intel RealSense D455 (87 x 58 deg FOV), which matches the
        90 deg / 8 m sensor configured for it and is the D400-series part
-       normally fitted to a mobile base. Mesh referenced out of
-       realsense2_description, not copied.
+       normally fitted to a mobile base. Mesh vendored from
+       realsense2_description into meshes/sensors/.
        IT IS A D455 AND NOT A D435 FOR A RENDERING REASON, measured not assumed.
        Gazebo (gz-sim 8.14, ogre2) IGNORES an SDF <material> on a mesh that
@@ -338,5 +345,5 @@
       <origin xyz="0.00465 0 0" rpy="${PI/2} 0 ${PI/2}"/>
       <geometry>
-        <mesh filename="package://realsense2_description/meshes/d455.stl"
+        <mesh filename="package://pickplace_arm_description/meshes/sensors/d455.stl"
               scale="0.001 0.001 0.001"/>
       </geometry>
@@ -399,5 +406,5 @@
        built for exactly this eye-in-hand job (60 deg HFOV, useful from a few
        mm out), which matches the 60 deg / 0.05-5 m sensor configured for it.
-       Mesh referenced out of realsense2_description, not copied.
+       Mesh vendored from realsense2_description into meshes/sensors/.
        Offsets copied from Intel's _d405.urdf.xacro, same convention as the
        D435 above: mesh at (zero_depth_to_glass + glass_to_front, -cam_depth_py,
@@ -408,5 +415,5 @@
       <origin xyz="0.0038 -0.009 0" rpy="${PI/2} 0 ${PI/2}"/>
       <geometry>
-        <mesh filename="package://realsense2_description/meshes/d405.stl"
+        <mesh filename="package://pickplace_arm_description/meshes/sensors/d405.stl"
               scale="0.001 0.001 0.001"/>
       </geometry>
